Commit message: added mapping config, changes to the TF tree and updated the robot bringup launch

File: description/robot_core.xacro (robot description, xacro)
@@ -18,4 +18,11 @@
   <link name="base_link">
   </link>
+  <link name="base_footprint">
+  </link>
+  <joint name="base_footprint_joint" type="fixed">
+      <parent link="base_link"/>
+      <child link="base_footprint"/>
+      <origin xyz="0 0 0" rpy="0 0 0"/>
+  </joint>
   <joint name="chassis_joint" type="fixed">
       <parent link="base_link"/>
