Commit message: added micro-ros agent, added basic nav2 mapping

File: description/robot.urdf.xacro (robot description, xacro)
@@ -4,4 +4,4 @@
    <xacro:include filename="ros2_control.xacro" />
    <xacro:include filename="lidar.xacro" />
-   <xacro:include filename="depth_sensor.xacro" />
+   <!--<xacro:include filename="depth_sensor.xacro" /> -->
 </robot>

File: description/robot_core.xacro (robot description, xacro)
@@ -32,14 +32,14 @@
   <link name="chassis">
       <visual>
-          <origin xyz="0.152 0 0.03" rpy="0 0 0"/>
+          <origin xyz="0.152 0 0.031" rpy="0 0 0"/>
           <geometry>
-              <box size="0.322 0.304 0.06"/>
+              <box size="0.332 0.304 0.06"/>
           </geometry>
           <material name="green"/>
       </visual>
       <collision>
-        <origin xyz="0.152 0 0.03" rpy="0 0 0"/>
+        <origin xyz="0.152 0 0.031" rpy="0 0 0"/>
         <geometry>
-            <box size="0.304 0.322 0.06"/>
+            <box size="0.304 0.332 0.06"/>
         </geometry>
       </collision>
@@ -49,5 +49,5 @@
       <parent link="base_link"/>
       <child link="left_wheel"/>
-      <origin xyz="0 0.131 0.017" rpy="-${pi/2} 0 0"/>
+      <origin xyz="0 0.131 0.0" rpy="-${pi/2} 0 0"/>
       <axis xyz="0 0 1"/>
   </joint>
@@ -55,5 +55,5 @@
       <visual>
           <geometry>
-              <cylinder length="0.03" radius="0.0325" />
+              <cylinder length="0.04" radius="0.044" />
           </geometry>
           <material name="black"/>
@@ -61,5 +61,5 @@
       <collision>
           <geometry>
-              <cylinder length="0.03" radius="0.0325" />
+              <cylinder length="0.04" radius="0.044" />
           </geometry>
       </collision>
@@ -69,5 +69,5 @@
       <parent link="base_link"/>
       <child link="right_wheel"/>
-      <origin xyz="0 -0.131 0.017" rpy="${pi/2} 0 0"/>
+      <origin xyz="0 -0.131 0.0" rpy="${pi/2} 0 0"/>
       <axis xyz="0 0 -1"/>
   </joint>
@@ -75,5 +75,5 @@
       <visual>
           <geometry>
-              <cylinder length="0.03" radius="0.0325" />
+              <cylinder length="0.04" radius="0.044" />
           </geometry>
           <material name="black"/>
@@ -81,5 +81,5 @@
       <collision>
           <geometry>
-              <cylinder length="0.03" radius="0.0325" />
+              <cylinder length="0.04" radius="0.044" />
           </geometry>
       </collision>
