Commit message: updated robot description and added new hardware script for fan and headlight contol

File: description/lidar.xacro (robot description, xacro)
@@ -4,5 +4,5 @@
         <parent link="chassis"/>
         <child link="laser_frame"/>
-        <origin xyz="0.267 0.075 0.08" rpy="0 0 ${pi/2}"/>
+        <origin xyz="0.267 0.1025 0.08" rpy="0 0 ${pi/2}"/>
     </joint>
     <link name="laser_frame">

File: description/robot_core.xacro (robot description, xacro)
@@ -34,5 +34,5 @@
           <origin xyz="0.152 0 0.031" rpy="0 0 0"/>
           <geometry>
-              <box size="0.332 0.304 0.06"/>
+              <box size="0.322 0.304 0.06"/>
           </geometry>
           <material name="green"/>
@@ -41,5 +41,5 @@
         <origin xyz="0.152 0 0.031" rpy="0 0 0"/>
         <geometry>
-            <box size="0.304 0.332 0.06"/>
+            <box size="0.322 0.304 0.06"/>
         </geometry>
       </collision>
@@ -49,5 +49,5 @@
       <parent link="base_link"/>
       <child link="left_wheel"/>
-      <origin xyz="0 0.131 0.0" rpy="-${pi/2} 0 0"/>
+      <origin xyz="0 0.125 0.005" rpy="-${pi/2} 0 0"/>
       <axis xyz="0 0 1"/>
   </joint>
@@ -55,5 +55,5 @@
       <visual>
           <geometry>
-              <cylinder length="0.04" radius="0.044" />
+              <cylinder length="0.04" radius="0.042" />
           </geometry>
           <material name="black"/>
@@ -61,5 +61,5 @@
       <collision>
           <geometry>
-              <cylinder length="0.04" radius="0.044" />
+              <cylinder length="0.04" radius="0.042" />
           </geometry>
       </collision>
@@ -69,5 +69,5 @@
       <parent link="base_link"/>
       <child link="right_wheel"/>
-      <origin xyz="0 -0.131 0.0" rpy="${pi/2} 0 0"/>
+      <origin xyz="0 -0.125 0.005" rpy="${pi/2} 0 0"/>
       <axis xyz="0 0 -1"/>
   </joint>
@@ -75,5 +75,5 @@
       <visual>
           <geometry>
-              <cylinder length="0.04" radius="0.044" />
+              <cylinder length="0.04" radius="0.042" />
           </geometry>
           <material name="black"/>
@@ -81,5 +81,5 @@
       <collision>
           <geometry>
-              <cylinder length="0.04" radius="0.044" />
+              <cylinder length="0.04" radius="0.042" />
           </geometry>
       </collision>

Commit message: latest changes

File: description/lidar.xacro (robot description, xacro)
@@ -4,6 +4,7 @@
         <parent link="chassis"/>
         <child link="laser_frame"/>
-        <origin xyz="0.267 0.1025 0.08" rpy="0 0 ${pi/2}"/>
+        <origin xyz="0.267 0.0575 0.08" rpy="0 0 ${pi/2}"/>
     </joint>
+    <!-- 0.1025 -->
     <link name="laser_frame">
         <visual>
