Commit message: Added depth camera functionality

File: description/depth_sensor.xacro (robot description, xacro)
@@ -5,5 +5,5 @@
         <parent link="chassis"/>
         <child link="camera_link"/>
-        <origin xyz="0.3 0.06 0.055" rpy="0 0 0"/>
+        <origin xyz="0.3 0.0 0.055" rpy="0 0 0"/>
     </joint>
     <link name="camera_link">

File: description/robot.urdf.xacro (robot description, xacro)
@@ -4,4 +4,4 @@
    <xacro:include filename="ros2_control.xacro" />
    <xacro:include filename="lidar.xacro" />
-   <!--<xacro:include filename="depth_sensor.xacro" /> -->
+   <xacro:include filename="depth_sensor.xacro" />
 </robot>

File: description/robot_core.xacro (robot description, xacro)
@@ -34,5 +34,5 @@
           <origin xyz="0.152 0 0.031" rpy="0 0 0"/>
           <geometry>
-              <box size="0.322 0.304 0.06"/>
+              <box size="0.322 0.304 0.1"/>
           </geometry>
           <material name="green"/>
@@ -41,5 +41,5 @@
         <origin xyz="0.152 0 0.031" rpy="0 0 0"/>
         <geometry>
-            <box size="0.322 0.304 0.06"/>
+            <box size="0.322 0.304 0.1"/>
         </geometry>
       </collision>
